File: NixieDisplayBoard/NixieDisplayBoard.sch (KiCad schematic (older format))
At the start: 4 parts, among them P1 CONN_01X12, P2 CONN_01X12

Commit message: Makes the nixie breakout board less stupid about which pins mean what...
Connections:
- net at N1.0: now also P1.2 (P2); no longer P1.12 (P12)
- net at N1.1: now also P1.3 (P3); no longer P1.10 (P10)
- net at N1.2: now also P1.4 (P4); no longer P1.9 (P9)
- net at N1.3: now also P1.5 (P5); no longer P1.8 (P8)
- net at N1.4: now also P1.6 (P6); no longer P1.7 (P7)
- net at N1.5: now also P1.7 (P7); no longer P1.6 (P6)
- net at N1.6: now also P1.8 (P8); no longer P1.5 (P5)
- net at N1.7: now also P1.9 (P9); no longer P1.4 (P4)
- net at N1.8: now also P1.10 (P10); no longer P1.3 (P3)
- net at N1.9: now also P1.11 (P11); no longer P1.2 (P2)
- net at N1.LHDP: now also P1.12 (P12); no longer P1.11 (P11)
- net at N2.0: now also P2.2 (P2); no longer P2.12 (P12)
- net at N2.1: now also P2.3 (P3); no longer P2.10 (P10)
- net at N2.2: now also P2.4 (P4); no longer P2.9 (P9)
- net at N2.3: now also P2.5 (P5); no longer P2.8 (P8)
- net at N2.4: now also P2.6 (P6); no longer P2.7 (P7)
- net at N2.5: now also P2.7 (P7); no longer P2.6 (P6)
- net at N2.6: now also P2.8 (P8); no longer P2.5 (P5)
- net at N2.7: now also P2.9 (P9); no longer P2.4 (P4)
- net at N2.8: now also P2.10 (P10); no longer P2.3 (P3)
- net at N2.9: now also P2.11 (P11); no longer P2.2 (P2)
- net at N2.LHDP: now also P2.12 (P12); no longer P2.11 (P11)
Changed lines of the file:
@@
 LIBS:contrib
 LIBS:valves
-LIBS:NixieComponentLibrary
-LIBS:russian-nixies
 LIBS:NixieDisplayBoard-cache
 EELAYER 25 0
@@
 $EndComp
 Wire Wire Line
-	5950 1150 5950 1000
-Wire Wire Line
-	5950 1000 5500 1000
-Wire Wire Line
-	5500 1000 5500 2400
-Wire Wire Line
-	5500 2400 6400 2400
-Wire Wire Line
-	6400 2400 6400 2250
-Wire Wire Line
-	5950 1250 6100 1250
-Wire Wire Line
-	6100 1250 6100 900
-Wire Wire Line
-	6100 900  7300 900
+	5950 2250 5950 2550
+Wire Wire Line
+	5950 2550 7300 2550
+Wire Wire Line
+	7300 2550 7300 1850
+Wire Wire Line
+	5950 3950 5950 4250
+Wire Wire Line
+	5950 4250 7300 4250
+Wire Wire Line
+	7300 4250 7300 3550
+Wire Wire Line
+	5950 3850 6050 3850
+Wire Wire Line
+	6050 3850 6050 3950
+Wire Wire Line
+	6050 3950 6400 3950
+Wire Wire Line
+	5950 3750 6350 3750
+Wire Wire Line
+	6350 3750 6350 3050
+Wire Wire Line
+	6350 3050 6400 3050
+Wire Wire Line
+	5950 3650 6300 3650
+Wire Wire Line
+	6300 3650 6300 3150
+Wire Wire Line
+	6300 3150 6400 3150
+Wire Wire Line
+	5950 3550 6250 3550
+Wire Wire Line
+	6250 3550 6250 3250
+Wire Wire Line
+	6250 3250 6400 3250
+Wire Wire Line
+	5950 3450 6200 3450
+Wire Wire Line
+	6200 3450 6200 3350
+Wire Wire Line
+	6200 3350 6400 3350
+Wire Wire Line
+	5950 3350 6150 3350
+Wire Wire Line
+	6150 3350 6150 3500
+Wire Wire Line
+	6150 3500 6400 3500
+Wire Wire Line
+	6400 3500 6400 3450
+Wire Wire Line
+	5950 3250 6100 3250
+Wire Wire Line
+	6100 3250 6100 3600
+Wire Wire Line
+	6100 3600 6400 3600
+Wire Wire Line
+	6400 3600 6400 3550
+Wire Wire Line
+	5950 3150 6050 3150
+Wire Wire Line
+	6050 3150 6050 3700
+Wire Wire Line
+	6050 3700 6400 3700
+Wire Wire Line
+	6400 3700 6400 3650
+Wire Wire Line
+	5950 3050 6000 3050
+Wire Wire Line
+	6000 3050 6000 3800
+Wire Wire Line
+	6000 3800 6400 3800
+Wire Wire Line
+	6400 3800 6400 3750
+Wire Wire Line
+	5950 2950 5950 3900
+Wire Wire Line
+	5950 3900 6400 3900
+Wire Wire Line
+	6400 3900 6400 3850
+Wire Wire Line
+	5950 2850 5950 2700
+Wire Wire Line
+	5950 2700 7300 2700
+Wire Wire Line
+	7300 2700 7300 3050
+Wire Wire Line
+	5950 2150 5950 2200
+Wire Wire Line
+	5950 2200 6400 2200
+Wire Wire Line
+	6400 2200 6400 2250
+Wire Wire Line
+	5950 2050 6350 2050
+Wire Wire Line
+	6350 2050 6350 1350
+Wire Wire Line
+	6350 1350 6400 1350
+Wire Wire Line
+	5950 1950 6300 1950
+Wire Wire Line
+	6300 1950 6300 1450
+Wire Wire Line
+	6300 1450 6400 1450
+Wire Wire Line
+	5950 1850 6250 1850
+Wire Wire Line
+	6250 1850 6250 1550
+Wire Wire Line
+	6250 1550 6400 1550
+Wire Wire Line
+	5950 1750 6200 1750
+Wire Wire Line
+	6200 1750 6200 1650
+Wire Wire Line
+	6200 1650 6400 1650
+Wire Wire Line
+	5950 1650 6150 1650
+Wire Wire Line
+	6150 1650 6150 1700
+Wire Wire Line
+	6150 1700 6400 1700
+Wire Wire Line
+	6400 1700 6400 1750
+Wire Wire Line
+	5950 1550 6100 1550
+Wire Wire Line
+	6100 1550 6100 1800
+Wire Wire Line
+	6100 1800 6400 1800
+Wire Wire Line
+	6400 1800 6400 1850
+Wire Wire Line
+	5950 1450 6050 1450
+Wire Wire Line
+	6050 1450 6050 1900
+Wire Wire Line
+	6050 1900 6400 1900
+Wire Wire Line
+	6400 1900 6400 1950
+Wire Wire Line
+	5950 1350 6000 1350
+Wire Wire Line
+	6000 1350 6000 2000
+Wire Wire Line
+	6000 2000 6400 2000
+Wire Wire Line
+	6400 2000 6400 2050
+Wire Wire Line
+	5950 1250 5950 2100
+Wire Wire Line
+	5950 2100 6400 2100
+Wire Wire Line
+	6400 2100 6400 2150
+Wire Wire Line
+	5950 1150 5950 900
+Wire Wire Line
+	5950 900  7300 900
 Wire Wire Line
 	7300 900  7300 1350
-Wire Wire Line
-	5950 2850 5950 2700
-Wire Wire Line
-	5950 2700 5500 2700
-Wire Wire Line
-	5500 2700 5500 4100
-Wire Wire Line
-	5500 4100 6400 4100
-Wire Wire Line
-	6400 4100 6400 3950
-Wire Wire Line
-	5950 2950 6100 2950
-Wire Wire Line
-	6100 2950 6100 2600
-Wire Wire Line
-	6100 2600 7300 2600
-Wire Wire Line
-	7300 2600 7300 3050
-Wire Wire Line
-	5950 3050 6400 3050
-Wire Wire Line
-	5950 3150 6400 3150
-Wire Wire Line
-	5950 3250 6400 3250
-Wire Wire Line
-	5950 3350 6400 3350
-Wire Wire Line
-	5950 3450 6400 3450
-Wire Wire Line
-	5950 3550 6400 3550
-Wire Wire Line
-	5950 3650 6400 3650
-Wire Wire Line
-	5950 3750 6400 3750
-Wire Wire Line
-	5950 3850 6400 3850
-Wire Wire Line
-	5950 1350 6400 1350
-Wire Wire Line
-	5950 1450 6400 1450
-Wire Wire Line
-	5950 1550 6400 1550
-Wire Wire Line
-	5950 1650 6400 1650
-Wire Wire Line
-	5950 1750 6400 1750
-Wire Wire Line
-	5950 1850 6400 1850
-Wire Wire Line
-	5950 1950 6400 1950
-Wire Wire Line
-	5950 2050 6400 2050
-Wire Wire Line
-	5950 2150 6400 2150
-Wire Wire Line
-	5950 2250 5950 2550
-Wire Wire Line
-	5950 2550 7300 2550
-Wire Wire Line
-	7300 2550 7300 1850
-Wire Wire Line
-	5950 3950 5950 4250
-Wire Wire Line
-	5950 4250 7300 4250
-Wire Wire Line
-	7300 4250 7300 3550
 $EndSCHEMATC
